Commit message: update

File: assets/urdf/dobot_l20/dobot_right_l20.urdf (robot description, URDF)
Before this commit: robot cr5_robot, 30 links, 29 joints
Joints:
- removed joint joint1
- removed joint joint2
- removed joint joint3
- removed joint joint4
- removed joint joint5
- removed joint joint6
- added joint dobot_joint_1: type revolute, parent base_link, child Link1, origin xyz=0 0 0.147 rpy=0 0 0, axis 0 0 1, limit lower=-6.28 upper=6.28 effort=300 velocity=10
- added joint dobot_joint_2: type revolute, parent Link1, child Link2, origin xyz=0 0 0 rpy=1.5708 1.5708 0, axis 0 0 1, limit lower=-6.28 upper=6.28 effort=300 velocity=10
- added joint dobot_joint_3: type revolute, parent Link2, child Link3, origin xyz=-0.427 0 0 rpy=0 0 0, axis 0 0 1, limit lower=-6.28 upper=6.28 effort=300 velocity=10
- added joint dobot_joint_4: type revolute, parent Link3, child Link4, origin xyz=-0.357 0 0.141 rpy=0 0 -1.5708, axis 0 0 1, limit lower=-6.28 upper=6.28 effort=300 velocity=10
- added joint dobot_joint_5: type revolute, parent Link4, child Link5, origin xyz=0 -0.116 0 rpy=1.5708 0 0, axis 0 0 1, limit lower=-6.28 upper=6.28 effort=300 velocity=10
- added joint dobot_joint_6: type revolute, parent Link5, child Link6, origin xyz=0 0.1 0 rpy=-1.5708 0 0, axis 0 0 1, limit lower=-6.28 upper=6.28 effort=300 velocity=10

File: assets/urdf/table_narrow.urdf (robot description, URDF)
Before this commit: robot box, 1 links, 0 joints
Links:
- link box: geometry collision box size=0.475 0.4 0.3; visual box size=0.475 0.4 0.3
