Commit message: update

File: assets/urdf/realman/rm_75b_left_sharpa.urdf (robot description, URDF)
Before this commit: robot rm_75_6f_description, 43 links, 42 joints
Joints:
- joint rm75b_joint_7: origin xyz=0 0 0.067 rpy=0 0 0 -> xyz=0 0 0.1728 rpy=0 0 0
- joint rm75b_joint_ee: origin xyz=0 0 0.0 rpy=0 0 0 -> xyz=0 0 -0.05 rpy=0 0 0
